Commit message: ...

File: barrett_control/barrett_model/models/arm.urdf.xacro (robot description, xacro)
@@ -26,26 +26,4 @@
   <xacro:include filename="$(find barrett_model)/models/common.urdf.xacro"/>
   <xacro:include filename="$(find barrett_model)/models/components.urdf.xacro"/>
-  <xacro:macro name="wam_7dof" params="prefix parent_link xyz rpy">
-    <xacro:wam prefix="${prefix}" parent_link="${parent_link}" xyz="${xyz}" rpy="${rpy}"/>
-    <xacro:wam_wrist_left prefix="${prefix}"/>
-    <xacro:wam_wrist_palm_stump prefix="${prefix}"/>
-  </xacro:macro>
-  <xacro:macro name="wam_4dof" params="prefix parent_link xyz rpy">
-    <xacro:wam prefix="${prefix}" parent_link="${parent_link}" xyz="${xyz}" rpy="${rpy}"/>
-    <xacro:wam_stump prefix="${prefix}"/>
-  </xacro:macro>
-  <!-- upper arm only -->
-  <xacro:macro name="wam" params="prefix parent_link xyz rpy">
-    <xacro:wam_base prefix="${prefix}" parent_link="${parent_link}" xyz="${xyz}" rpy="${rpy}"/>
-    <xacro:wam_shoulder_yaw prefix="${prefix}" rpy="0 0 ${PI/2}" />
-    <xacro:wam_shoulder_pitch prefix="${prefix}" rpy="-${PI/2} ${PI/2} 0"/>
-    <xacro:wam_upper_arm prefix="${prefix}"/>
-  </xacro:macro>
-  <xacro:macro name="wam_right" params="prefix parent_link xyz rpy">
-    <xacro:wam_base prefix="${prefix}" parent_link="${parent_link}" xyz="${xyz}" rpy="${rpy}"/>
-    <xacro:wam_shoulder_yaw prefix="${prefix}" rpy="0 0 0" />
-    <xacro:wam_shoulder_pitch prefix="${prefix}" rpy="0 0 0"/>
-    <xacro:wam_upper_arm prefix="${prefix}" rpy="0 0 0"/>
-  </xacro:macro>
   <xacro:macro name="wam_left" params="prefix parent_link xyz rpy">
     <xacro:wam_base prefix="${prefix}" parent_link="${parent_link}" xyz="${xyz}" rpy="${rpy}"/>
@@ -56,8 +34,10 @@
   <!-- forearm with actuation "wrist" -->
   <xacro:macro name="wam_wrist_right" params="prefix">
-    <xacro:wam_forearm prefix="${prefix}"/>
+    <!-- <xacro:wam_forearm prefix="${prefix}"/> -->
+    <!--
     <xacro:wam_wrist_yaw prefix="${prefix}" rpy="${PI/2} 0 0"/>
     <xacro:wam_wrist_pitch prefix="${prefix}"/>
     <xacro:wam_palm prefix="${prefix}" rpy="${PI/2} -${PI/2} 0"/>
+    -->
   </xacro:macro>
   <xacro:macro name="wam_wrist_left" params="prefix">

File: barrett_control/barrett_model/models/components.urdf.xacro (robot description, xacro)
@@ -24,7 +24,9 @@
 -->
 <robot xmlns:xacro="http://ros.org/wiki/xacro">
-  <xacro:include filename="$(find barrett_model)/models/hand.urdf.xacro"/>
+  <!-- <xacro:include filename="$(find barrett_model)/models/hand.urdf.xacro"/> -->
   <xacro:include filename="$(find barrett_model)/models/common.urdf.xacro"/>
   <xacro:property name="b" value="0.5"/>
+  <xacro:include filename="$(find barrett_model)/robots/wam7_bhand.transmission.xacro"/>
+  <xacro:include filename="$(find barrett_model)/robots/wam7_bhand.gazebo.xacro"/>
   <!-- Upper arm macros -->
   <xacro:macro name="wam_base" params="prefix parent_link xyz rpy">
@@ -49,4 +51,5 @@
         <geometry>
           <mesh filename="${models_path}/sw_meshes/base_link_convex.dae"/>
+          <!-- <mesh filename="package://barrett_model/meshes/wambase.stl" /> -->
         </geometry>
       </visual>
@@ -54,4 +57,5 @@
         <geometry>
           <mesh filename="${models_path}/sw_meshes/base_link_convex.dae"/>
+          <!-- <mesh filename="package://barrett_model/meshes/wambase.stl" /> -->
         </geometry>
       </collision>
@@ -64,5 +68,5 @@
       <origin xyz="0 0 0.346" rpy="${rpy}"/>
       <axis xyz="0 0 1"/>
-      <limit effort="60" lower="-2.6" upper="2.6" velocity="2.0"/>
+      <limit effort="25" lower="-2.6" upper="2.6" velocity="2.0"/>
       <dynamics damping="${1.8*b}" friction="0"/>
     </joint>
@@ -85,4 +89,5 @@
         <geometry>
           <mesh filename="${models_path}/sw_meshes/shoulder_link_convex_decomposition.dae"/>
+          <!-- <mesh filename="package://barrett_model/meshes/wam1.stl" /> -->
         </geometry>
       </visual>
@@ -90,4 +95,5 @@
         <geometry>
           <mesh filename="${models_path}/sw_meshes/shoulder_link_convex_decomposition.dae"/>
+          <!-- <mesh filename="package://barrett_model/meshes/wam1.stl" /> -->
         </geometry>
       </collision>
@@ -98,7 +104,7 @@
       <parent link="${prefix}/shoulder_yaw_link"/>
       <child link="${prefix}/shoulder_pitch_link"/>
-      <origin xyz="0 0 0" rpy="${rpy}"/>
-      <axis xyz="0 1 0"/>
-      <limit effort="60" lower="-2.0" upper="2.0" velocity="2.0"/>
+      <origin xyz="0 0 0" rpy="${-PI/2} 0 0"/>
+      <axis xyz="0 0 1"/>
+      <limit effort="20" lower="-2.0" upper="2.0" velocity="2.0"/>
       <dynamics damping="${0.5*b}" friction="0"/>
     </joint>
@@ -113,4 +119,5 @@
         <geometry>
           <mesh filename="${models_path}/sw_meshes/shoulder_pitch_link_convex.dae"/>
+          <!-- <mesh filename="package://barrett_model/meshes/wam2.stl" /> -->
         </geometry>
       </visual>
@@ -126,4 +133,5 @@
         <geometry>
           <mesh filename="${models_path}/sw_meshes/shoulder_pitch_link_convex.dae"/>
+          <!-- <mesh filename="package://barrett_model/meshes/wam2.stl" /> -->
         </geometry>
       </collision>
@@ -134,7 +142,7 @@
       <parent link="${prefix}/shoulder_pitch_link"/>
       <child link="${prefix}/upper_arm_link"/>
-      <origin xyz="0 0 0" rpy="${rpy}"/>
-      <axis xyz="0 0 1"/>
-      <limit effort="45" lower="-2.8" upper="2.8" velocity="2.0"/>
+      <origin xyz="0 0 0" rpy="${PI/2} 0 0"/>
+      <axis xyz="0 0 1"/>
+      <limit effort="15" lower="-2.8" upper="2.8" velocity="2.0"/>
       <dynamics damping="${1.5*b}" friction="0"/>
     </joint>
@@ -157,4 +165,5 @@
         <geometry>
           <mesh filename="${models_path}/sw_meshes/upper_arm_link_convex_decomposition.dae"/>
+          <!-- <mesh filename="package://barrett_model/meshes/wam3.stl" /> -->
         </geometry>
       </visual>
@@ -162,4 +171,5 @@
         <geometry>
           <mesh filename="${models_path}/sw_meshes/upper_arm_link_convex_decomposition.dae"/>
+          <!-- <mesh filename="package://barrett_model/meshes/wam3.stl" /> -->
         </geometry>
       </collision>
@@ -173,5 +183,5 @@
       <origin xyz="0.045 0 0.55" rpy="${-PI/2} 0 0"/>
       <axis xyz="0 0 1"/>
-      <limit effort="30" lower="-0.9" upper="${PI}" velocity="2.00"/>
+      <limit effort="15" lower="-0.9" upper="${PI}" velocity="2.00"/>
       <dynamics damping="${0.8*b}" friction="0"/>
     </joint>
@@ -194,4 +204,5 @@
         <geometry>
           <mesh filename="${models_path}/sw_meshes/elbow_link_convex.dae"/>
+          <!-- <mesh filename="package://barrett_model/meshes/wam4.stl" /> -->
         </geometry>
       </visual>
@@ -199,4 +210,5 @@
         <geometry>
           <mesh filename="${models_path}/sw_meshes/elbow_link_convex.dae"/>
+          <!-- <mesh filename="package://barrett_model/meshes/wam4.stl" /> -->
         </geometry>
       </collision>
@@ -224,5 +236,5 @@
       <origin xyz="-0.045 -0.3 0" rpy="${rpy}"/>
       <axis xyz="0 0 1"/>
-      <limit effort="10" lower="-4.76" upper="1.24" velocity="2.0"/>
+      <limit effort="5" lower="-4.76" upper="1.24" velocity="2.0"/>
       <dynamics damping="${0.5*b}" friction="0"/>
     </joint>
@@ -245,4 +257,5 @@
         <geometry>
           <mesh filename="${models_path}/sw_meshes/wrist_yaw_link_convex_decomposition.dae"/>
+          <!-- <mesh filename="package://barrett_model/meshes/wam5.stl" /> -->
         </geometry>
       </visual>
@@ -251,4 +264,5 @@
         <geometry>
           <mesh filename="${models_path}/sw_meshes/wrist_yaw_link_convex_decomposition.dae"/>
+          <!-- <mesh filename="package://barrett_model/meshes/wam5.stl" /> -->
         </geometry>
       </collision>
@@ -261,5 +275,5 @@
       <origin xyz="0 0 0" rpy="${-PI/2} 0 0"/>
       <axis xyz="0 0 1"/>
-      <limit effort="10" lower="-1.6" upper="1.6" velocity="2.00"/>
+      <limit effort="5" lower="-1.6" upper="1.6" velocity="2.00"/>
       <dynamics damping="${0.1*b}" friction="0"/>
     </joint>
@@ -282,4 +296,5 @@
         <geometry>
           <mesh filename="${models_path}/sw_meshes/wrist_pitch_link_convex_decomposition.dae"/>
+          <!-- <mesh filename="package://barrett_model/meshes/wam6.stl" /> -->
         </geometry>
       </visual>
@@ -287,4 +302,5 @@
         <geometry>
           <mesh filename="${models_path}/sw_meshes/wrist_pitch_link_convex_decomposition.dae"/>
+          <!-- <mesh filename="package://barrett_model/meshes/wam6.stl" /> -->
         </geometry>
       </collision>
@@ -296,7 +312,7 @@
       <parent link="${prefix}/wrist_pitch_link"/>
       <child link="${prefix}/wrist_palm_link"/>
-      <origin xyz="0 0 0" rpy="${rpy}"/>
-      <axis xyz="0 0 1"/>
-      <limit effort="10" lower="-3.0" upper="3.0" velocity="2.00"/><!-- 2.95 is a limit taken in from 3 due to saftey and differences between arms. -->
+      <origin xyz="0 0 0" rpy="${PI/2} 0 0"/>
+      <axis xyz="0 0 1"/>
+      <limit effort="5" lower="-3.0" upper="3.0" velocity="2.00"/><!-- 2.95 is a limit taken in from 3 due to saftey and differences between arms. -->
       <dynamics damping="${0.1*b}" friction="0"/>
     </joint>
@@ -319,4 +335,5 @@
         <geometry>
           <mesh filename="${models_path}/sw_meshes/wrist_palm_link_convex.dae"/>
+          <!--<mesh filename="package://barrett_model/meshes/wam7.stl" /> -->
         </geometry>
       </visual>
@@ -325,4 +342,5 @@
         <geometry>
           <mesh filename="${models_path}/sw_meshes/wrist_palm_link_convex.dae"/>
+          <!-- <mesh filename="package://barrett_model/meshes/wam7.stl" /> -->
         </geometry>
       </collision>
@@ -371,5 +389,5 @@
         <!--<origin xyz="0 0 0" rpy="-${PI} 0 0" />-->
         <!--<geometry>-->
-          <!--<mesh filename="${models_path}/meshes/wamForeArmLink4.DAE"/>-->
+          <!--<mesh filename="${models_path}/meshes/wamForeArmLink4.dae"/>-->
         <!--</geometry>-->
       <!--</visual>-->
@@ -377,5 +395,5 @@
         <!--<origin xyz="0 0 0" rpy="-${PI} 0 0" />-->
         <!--<geometry>-->
-          <!--<mesh filename="${models_path}/meshes/wamForeArmLink4.stl"/>-->
+          <!--<mesh filename="${models_path}/meshes/wamForeArmLink4.dae"/>-->
         <!--</geometry>-->
       <!--</collision>-->
@@ -406,5 +424,5 @@
         <!--<origin xyz="0 0.02711 0" rpy="${PI} 0 0" />-->
         <!--<geometry>-->
-          <!--<mesh filename="${models_path}/meshes/wamUpperWristYawLink.DAE"/>-->
+          <!--<mesh filename="${models_path}/meshes/wamUpperWristYawLink.dae"/>-->
         <!--</geometry>-->
       <!--</visual>-->
@@ -412,5 +430,5 @@
         <!--<origin xyz="0 0.02711 0" rpy="${PI} 0 0" />-->
         <!--<geometry>-->
-          <!--<mesh filename="${models_path}/meshes/wamUpperWristYawLink5.stl"/>-->
+          <!--<mesh filename="${models_path}/meshes/wamUpperWristYawLink5.dae"/>-->
         <!--</geometry>-->
       <!--</collision>-->
@@ -442,5 +460,5 @@
         <!--<origin xyz="0 0 0" rpy="0 0 0" />-->
         <!--<geometry>-->
-          <!--<mesh filename="${models_path}/meshes/forceTorqueSensor.DAE"/>-->
+          <!--<mesh filename="${models_path}/meshes/forceTorqueSensor.dae"/>-->
         <!--</geometry>-->
       <!--</visual>-->
@@ -448,5 +466,5 @@
         <!--<origin xyz="0 0 0" rpy="0 0 0" />-->
         <!--<geometry>-->
-          <!--<mesh filename="${models_path}/meshes/forceTorqueSensor.stl"/>-->
+          <!--<mesh filename="${models_path}/meshes/forceTorqueSensor.dae"/>-->
         <!--</geometry>-->
       <!--</collision>-->

File: barrett_control/barrett_model/models/wam_top.urdf.xacro (robot description, xacro)
@@ -9,7 +9,7 @@
   <xacro:include filename="$(find barrett_model)/models/components.urdf.xacro"/>
   <!-- Definitions for the barrett hand -->
-  <xacro:include filename="$(find barrett_model)/models/hand.urdf.xacro"/>
+  <!-- <xacro:include filename="$(find barrett_model)/models/hand.urdf.xacro"/> -->
   <!-- Definitions for the barrett ball -->
-  <xacro:include filename="$(find barrett_model)/models/ball.urdf.xacro"/>
+  <!-- <xacro:include filename="$(find barrett_model)/models/ball.urdf.xacro"/>-->
   <!-- Materials -->
   <material name="WAMGrey">

File: barrett_control/barrett_model/robots/wam7_bhand.urdf (robot description, URDF)
Before this commit: robot wam, 16 links, 15 joints
Links:
- removed link left_wam/wrist_palm_link
- removed link left_wam/wrist_pitch_link
- removed link left_wam/wrist_yaw_link
- added link world
- link left_wam_rack: mass None -> 1
- link rack1: mass None -> 1
- link rack2: mass None -> 1
- link rack3: mass None -> 1
- link rack4: mass None -> 1
- link rack5: mass None -> 1
- link rack6: mass None -> 1
- link right_wam_rack: mass None -> 1
Joints:
- removed joint left_wam/palm_yaw_joint
- removed joint left_wam/wrist_pitch_joint
- removed joint left_wam/wrist_yaw_joint
- added joint fixed: type fixed, parent world, child rack1
- joint left_wam/base_yaw_joint: limit lower=-2.6 upper=2.6 effort=60 velocity=2.0 -> lower=-2.6 upper=2.6 effort=25 velocity=2.0
- joint left_wam/elbow_pitch_joint: limit lower=-0.9 upper=3.14159265359 effort=30 velocity=2.00 -> lower=-0.9 upper=3.14159265359 effort=15 velocity=2.00
- joint left_wam/shoulder_pitch_joint: axis 0 1 0 -> 0 0 1; limit lower=-2.0 upper=2.0 effort=60 velocity=2.0 -> lower=-2.0 upper=2.0 effort=20 velocity=2.0; origin xyz=0 0 0 rpy=0 0 0 -> xyz=0 0 0 rpy=-1.57079632679 0 0
- joint left_wam/shoulder_yaw_joint: limit lower=-2.8 upper=2.8 effort=45 velocity=2.0 -> lower=-2.8 upper=2.8 effort=15 velocity=2.0; origin xyz=0 0 0 rpy=0 0 0 -> xyz=0 0 0 rpy=1.57079632679 0 0

File: barrett_control/barrett_model/robots/wam7_bhand.urdf.xacro (robot description, xacro)
@@ -4,7 +4,14 @@
   <!-- Includea all the WAM stuff -->
   <xacro:include filename="$(find barrett_model)/models/wam_top.urdf.xacro"/>
+  <xacro:include filename="$(find barrett_model)/robots/wam7_bhand.transmission.xacro"/>
+  <xacro:include filename="$(find barrett_model)/robots/wam7_bhand.gazebo.xacro"/>
   <!-- Root link is in the world frame-->
   <xacro:property name="width" value="0.0889" />
   <xacro:property name="height" value="0.0492125" />
+  <link name="world"/>
+  <joint name="fixed" type="fixed">
+    <parent link="world"/>
+    <child link="rack1"/>
+  </joint>
   <link name="rack1">
     <visual>
@@ -13,4 +20,12 @@
       </geometry>
     </visual>
+    <inertial>
+        <origin xyz="0 0 0" />
+        <mass value="1" />
+        <inertia
+          ixx="0.1" ixy="0"   ixz="0"
+                  iyy="0.1"   iyz="0"
+                            izz="0.1" />
+    </inertial>
   </link>
   <link name="rack2">
@@ -21,4 +36,12 @@
       <origin rpy="0 0 1.57075" xyz="0 0 0"/>
     </visual>
+    <inertial>
+        <origin xyz="0 0 0" />
+        <mass value="1" />
+        <inertia
+          ixx="0.1" ixy="0"   ixz="0"
+                  iyy="0.1"   iyz="0"
+                            izz="0.1" />
+    </inertial>
   </link>
   <link name="rack3">
@@ -29,4 +52,12 @@
       <origin rpy="0 0 1.57075" xyz="0 0 0"/>
     </visual>
+    <inertial>
+        <origin xyz="0 0 0" />
+        <mass value="1" />
+        <inertia
+          ixx="0.1" ixy="0"   ixz="0"
+                  iyy="0.1"   iyz="0"
+                            izz="0.1" />
+    </inertial>
   </link>
   <link name="rack4">
@@ -37,4 +68,12 @@
       <origin rpy="0 0 1.57075" xyz="0 0 0"/>
     </visual>
+    <inertial>
+        <origin xyz="0 0 0" />
+        <mass value="1" />
+        <inertia
+          ixx="0.1" ixy="0"   ixz="0"
+                  iyy="0.1"   iyz="0"
+                            izz="0.1" />
+    </inertial>
   </link>
   <link name="rack5">
@@ -45,4 +84,12 @@
       <origin rpy="0 1.57075 0" xyz="0 0 0.9525"/>
     </visual>
+    <inertial>
+        <origin xyz="0 0 0" />
+        <mass value="1" />
+        <inertia
+          ixx="0.1" ixy="0"   ixz="0"
+                  iyy="0.1"   iyz="0"
+                            izz="0.1" />
+      </inertial>
   </link>
   <link name="rack6">
@@ -53,7 +100,33 @@
       <origin rpy="0 0 0" xyz="0 0 0"/>
     </visual>
+    <inertial>
+        <origin xyz="0 0 0" />
+        <mass value="1" />
+        <inertia
+          ixx="0.1" ixy="0"   ixz="0"
+                  iyy="0.1"   iyz="0"
+                            izz="0.1" />
+    </inertial>
   </link>
-  <link name ="left_wam_rack" />
-  <link name ="right_wam_rack" />
+  <link name ="left_wam_rack">
+    <inertial>
+        <origin xyz="0 0 0" />
+        <mass value="1" />
+        <inertia
+          ixx="0.1" ixy="0"   ixz="0"
+                  iyy="0.1"   iyz="0"
+                            izz="0.1" />
+    </inertial>
+  </link>
+  <link name ="right_wam_rack">
+    <inertial>
+        <origin xyz="0 0 0" />
+        <mass value="1" />
+        <inertia
+          ixx="0.1" ixy="0"   ixz="0"
+                  iyy="0.1"   iyz="0"
+                            izz="0.1" />
+     </inertial>
+  </link>
   <joint name="rack1_to_rack2" type="fixed">
     <parent link="rack1"/>
@@ -100,3 +173,6 @@
   <xacro:wam_wrist_left prefix="left_wam"/>
   <!-- <xacro:bhand prefix="left_wam/bhand" parent_link="left_wam/wrist_palm_link" xyz="0 0 0.06" rpy="0 0 0"/> -->
+  <!-- gazebo stuff -->
+  <xacro:wam7_bhand_gazebo prefix="left_wam" name="barrett_hw"/>
+  <xacro:wam7_bhand_transmission prefix="left_wam" name="barrett_hw"/>
 </robot>
